Commit message: Removed front tires until confirmed working

File: mybot_description/urdf/mybot.xacro (robot description, xacro)
@@ -102,28 +102,4 @@
     </inertial>
   </link>
-  <link name="front_left_wheel">
-    <!--origin xyz="0.1 0.13 0.1" rpy="0 1.5707 1.5707"/-->
-    <collision name="collision">
-      <origin xyz="0 0 0" rpy="0 1.5707 1.5707"/>
-      <geometry>
-        <cylinder radius="0.1778" length="0.1524"/>
-      </geometry>
-    </collision>
-    <visual name="left_wheel_visual">
-      <origin xyz="0.0 0.0 0.0" rpy="0 1.5707 1.5707"/>
-      <geometry>
-        <mesh filename="package://mybot_description/meshes/Wheel.stl" scale="0.001 0.001 0.001"/>
-      </geometry>
-    </visual>
-    <inertial>
-      <origin xyz="0 0 0" rpy="0 1.5707 1.5707"/>
-      <mass value="5"/>
-      <cylinder_inertia m="5" r="0.1" h="0.05"/>
-      <inertia
-        ixx="0.004" ixy="0.001" ixz="0.0"
-        iyy="0.006" iyz="0.0"
-        izz="0.007"/>
-    </inertial>
-  </link>
   <joint type="continuous" name="left_wheel_hinge">
     <origin xyz="0.1 0.3 0" rpy="0 0 0"/>

Commit message: Added front right wheel to urdf
Need to add front left wheel to mybot.xacro and configure both front tires to turn, rather than drive forward

File: mybot_description/urdf/mybot.xacro (robot description, xacro)
@@ -102,6 +102,6 @@
     </inertial>
   </link>
-  <link name="front_left_wheel">
-    <!--origin xyz="0.1 0.13 0.1" rpy="0 1.5707 1.5707"/-->
+  <link name="front_right_wheel">
+    <!--origin xyz="0.1 -0.13 0.1" rpy="0 1.5707 1.5707"/-->
     <collision name="collision">
       <origin xyz="0 0 0" rpy="0 1.5707 1.5707"/>
@@ -110,6 +110,6 @@
       </geometry>
     </collision>
-    <visual name="left_wheel_visual">
-      <origin xyz="0.0 0.0 0.0" rpy="0 1.5707 1.5707"/>
+    <visual name="right_wheel_visual">
+      <origin xyz="0.0 0.0 0.0" rpy="1.57075 0 0"/>
       <geometry>
         <mesh filename="package://mybot_description/meshes/Wheel.stl" scale="0.001 0.001 0.001"/>
@@ -119,5 +119,5 @@
       <origin xyz="0 0 0" rpy="0 1.5707 1.5707"/>
       <mass value="5"/>
-      <cylinder_inertia m="5" r="0.1" h="0.05"/>
+      <!-- <cylinder_inertia m="5" r="0.1" h="0.05"/> -->
       <inertia
         ixx="0.004" ixy="0.001" ixz="0.0"
@@ -126,7 +126,7 @@
     </inertial>
   </link>
-  <joint type="continuous" name="left_wheel_hinge">
+  <joint type="continuous" name="back_left_wheel_hinge">
     <origin xyz="0.1 0.3 0" rpy="0 0 0"/>
-    <child link="left_wheel"/>
+    <child link="back_left_wheel"/>
     <parent link="chassis"/>
     <axis xyz="0 1 0" rpy="0 0 0"/>
@@ -134,7 +134,7 @@
     <joint_properties damping="0.0" friction="0.0"/>
   </joint>
-  <joint type="continuous" name="right_wheel_hinge">
+  <joint type="continuous" name="back_right_wheel_hinge">
     <origin xyz="0.1 -0.3 0" rpy="0 0 0"/>
-    <child link="right_wheel"/>
+    <child link="back_right_wheel"/>
     <parent link="chassis"/>
     <axis xyz="0 1 0" rpy="0 0 0"/>
@@ -142,4 +142,12 @@
     <joint_properties damping="0.0" friction="0.0"/>
   </joint>
+  <joint type="continuous" name="front_right_wheel_hinge">
+    <origin xyz="0.8 -0.3 0" rpy="0 0 0"/>
+    <child link="front_right_wheel"/>
+    <parent link="chassis"/>
+    <axis xyz="0 1 0" rpy="0 0 0"/>
+    <limit effort="100" velocity="100"/>
+    <joint_properties damping="0.0" friction="0.0"/>
+   </joint>
 <!--
   <link name="camera">

Commit message: Added front tires to vehicle but issues still occur
Updated to have both front tires but this creates a problem with the vehicle. In gazebo simulation the car flips out and it could be due to the arrangement of collisions

File: mybot_description/urdf/mybot.xacro (robot description, xacro)
@@ -17,13 +17,13 @@
       />
     </inertial>
-    <!--<collision name='collision'>
-      <origin xyz="0.0 -0.305 0.0" rpy=" 0 0 0"/>
-      <geometry>
-        <box size="1.143 0.700 0.27"/>
+    <collision name='collision'>
+      <origin xyz="0.36 0.3 0.45" rpy=" 0 0 0"/>
+      <geometry>
+        <box size="1.3 0.700 0.6"/>
       </geometry>
     </collision> -->
     <visual name='chassis_visual'>
             <!-- DO NOT CHANGE -->
-            <origin xyz="0.11 -0.3 0.02" rpy=" 1.5707 0.3066 0"/>
+            <origin xyz="0.0 0.0 0.2" rpy=" 1.5707 0.0 0"/>
       <geometry>
         <!-- <box size=".4 .2 .1"/> -->
@@ -31,27 +31,5 @@
       </geometry>
     </visual>
-    <collision name='caster_collision'>
-      <origin xyz="-0.15 0 -0.05" rpy=" 0 0 0"/>
-      <geometry>
-        <sphere radius="0.05"/>
-      </geometry>
-      <surface>
-        <friction>
-          <ode>
-            <mu>0</mu>
-            <mu2>0</mu2>
-            <slip1>1.0</slip1>
-            <slip2>1.0</slip2>
-          </ode>
-        </friction>
-      </surface>
-    </collision>
-    <visual name='caster_visual'>
-      <origin xyz="-0.15 0 -0.05" rpy=" 0 0 0"/>
-      <geometry>
-        <sphere radius="0.05"/>
-      </geometry>
-    </visual>
-  </link>
+   </link>
   <link name="back_left_wheel">
     <!--origin xyz="0.1 0.13 0.1" rpy="0 1.5707 1.5707"/-->
@@ -126,6 +104,30 @@
     </inertial>
   </link>
+  <link name="front_left_wheel">
+    <!--origin xyz="0.1 -0.13 0.1" rpy="0 1.5707 1.5707"/-->
+    <collision name="collision">
+      <origin xyz="0 0 0" rpy="0 1.5707 1.5707"/>
+      <geometry>
+        <cylinder radius="0.1778" length="0.1524"/>
+      </geometry>
+    </collision>
+    <visual name="left_wheel_visual">
+      <origin xyz="0.0 0.0 0.0" rpy="1.57075 0 0"/>
+      <geometry>
+        <mesh filename="package://mybot_description/meshes/Wheel.stl" scale="0.001 0.001 0.001"/>
+      </geometry>
+    </visual>
+    <inertial>
+      <origin xyz="0 0 0" rpy="0 1.5707 1.5707"/>
+      <mass value="5"/>
+      <!-- <cylinder_inertia m="5" r="0.1" h="0.05"/> -->
+      <inertia
+        ixx="0.004" ixy="0.001" ixz="0.0"
+        iyy="0.006" iyz="0.0"
+        izz="0.007"/>
+    </inertial>
+  </link>
   <joint type="continuous" name="back_left_wheel_hinge">
-    <origin xyz="0.1 0.3 0" rpy="0 0 0"/>
+    <origin xyz="0.1 0.8 0" rpy="0 0 0"/>
     <child link="back_left_wheel"/>
     <parent link="chassis"/>
@@ -135,5 +137,5 @@
   </joint>
   <joint type="continuous" name="back_right_wheel_hinge">
-    <origin xyz="0.1 -0.3 0" rpy="0 0 0"/>
+    <origin xyz="0.1 -0.8 0" rpy="0 0 0"/>
     <child link="back_right_wheel"/>
     <parent link="chassis"/>
@@ -143,5 +145,5 @@
   </joint>
   <joint type="continuous" name="front_right_wheel_hinge">
-    <origin xyz="0.8 -0.3 0" rpy="0 0 0"/>
+    <origin xyz="0.8 -0.8 0" rpy="0 0 0"/>
     <child link="front_right_wheel"/>
     <parent link="chassis"/>
@@ -149,4 +151,12 @@
     <limit effort="100" velocity="100"/>
     <joint_properties damping="0.0" friction="0.0"/>
+   </joint>
+   <joint type="continuous" name="front_left_wheel_hinge">
+     <origin xyz="0.8 0.0 0" rpy="0 0 0"/>
+     <child link="front_left_wheel"/>
+     <parent link="chassis"/>
+     <axis xyz="0 1 0" rpy="0 0 0"/>
+     <limit effort="100" velocity="100"/>
+     <joint_properties damping="0.0" friction="0.0"/>
    </joint>
 <!--

Commit message: Fixed laser and camera configuration

File: mybot_description/urdf/mybot.xacro (robot description, xacro)
@@ -9,24 +9,21 @@
     <pose>0 0 0.1 0 0 0</pose>
     <inertial>
-      <mass value="5.0"/>
-      <origin xyz="0.0 0.0 0.0" rpy="0 0 0"/>
+      <mass value="10.0"/>
+      <origin xyz="0.0 0 0.1" rpy=" 0 0 0"/>
       <inertia
-          ixx="0.004" ixy="0.001" ixz="0"
-          iyy="0.006" iyz="0"
-          izz="0.007"
+          ixx="0.5" ixy="0" ixz="0"
+          iyy="1.0" iyz="0"
+          izz="0.1"
       />
     </inertial>
-    <!--<collision name='collision'>
-      <origin xyz="0.0 -0.305 0.0" rpy=" 0 0 0"/>
+    <collision name='collision'>
       <geometry>
-        <box size="1.143 0.700 0.27"/>
+        <box size=".4 .2 .1"/>
       </geometry>
-    </collision> -->
+    </collision>
     <visual name='chassis_visual'>
-            <!-- DO NOT CHANGE -->
-            <origin xyz="0.11 -0.3 0.02" rpy=" 1.5707 0.3066 0"/>
+      <origin xyz="0 0 0" rpy=" 0 0 0"/>
       <geometry>
-        <!-- <box size=".4 .2 .1"/> -->
-        <mesh filename="package://mybot_description/meshes/JEEP.dae" scale="1 1 1"/>
+        <box size=".4 .2 .1"/>
       </geometry>
     </visual>
@@ -54,54 +51,54 @@
     </visual>
   </link>
-  <link name="back_left_wheel">
-    <!--origin xyz="0.1 0.13 0.1" rpy="0 1.5707 1.5707"/-->
-    <collision name="collision">
-      <origin xyz="0 0 0" rpy="0 1.5707 1.5707"/>
-      <geometry>
-        <cylinder radius="0.1778" length="0.1524"/>
-      </geometry>
-    </collision>
-    <visual name="left_wheel_visual">
-      <origin xyz="0.0 0.0 0.0" rpy="0 1.5707 1.5707"/>
-      <geometry>
-        <mesh filename="package://mybot_description/meshes/Wheel.stl" scale="0.001 0.001 0.001"/>
-      </geometry>
-    </visual>
-    <inertial>
-      <origin xyz="0 0 0" rpy="0 1.5707 1.5707"/>
-      <mass value="5"/>
-      <cylinder_inertia m="5" r="0.1" h="0.05"/>
-      <inertia
-        ixx="0.004" ixy="0.001" ixz="0.0"
-        iyy="0.006" iyz="0.0"
-        izz="0.007"/>
-    </inertial>
-  </link>
-  <link name="back_right_wheel">
-    <!--origin xyz="0.1 -0.13 0.1" rpy="0 1.5707 1.5707"/-->
-    <collision name="collision">
-      <origin xyz="0 0 0" rpy="0 1.5707 1.5707"/>
-      <geometry>
-        <cylinder radius="0.1778" length="0.1524"/>
-      </geometry>
-    </collision>
-    <visual name="right_wheel_visual">
-      <origin xyz="0.0 0.0 0.0" rpy="1.57075 0 0"/>
-      <geometry>
-        <mesh filename="package://mybot_description/meshes/Wheel.stl" scale="0.001 0.001 0.001"/>
-      </geometry>
-    </visual>
-    <inertial>
-      <origin xyz="0 0 0" rpy="0 1.5707 1.5707"/>
-      <mass value="5"/>
-      <!-- <cylinder_inertia m="5" r="0.1" h="0.05"/> -->
-      <inertia
-        ixx="0.004" ixy="0.001" ixz="0.0"
-        iyy="0.006" iyz="0.0"
-        izz="0.007"/>
-    </inertial>
-  </link>
+  <link name="left_wheel">
+      <!--origin xyz="0.1 0.13 0.1" rpy="0 1.5707 1.5707"/-->
+      <collision name="collision">
+        <origin xyz="0 0 0" rpy="0 1.5707 1.5707"/>
+        <geometry>
+          <cylinder radius="0.1" length="0.05"/>
+        </geometry>
+      </collision>
+      <visual name="left_wheel_visual">
+        <origin xyz="0 0 0" rpy="0 1.5707 1.5707"/>
+        <geometry>
+          <cylinder radius="0.1" length="0.05"/>
+        </geometry>
+      </visual>
+      <inertial>
+        <origin xyz="0 0 0" rpy="0 1.5707 1.5707"/>
+        <mass value="5"/>
+        <cylinder_inertia m="5" r="0.1" h="0.05"/>
+        <inertia
+          ixx="1.0" ixy="0.0" ixz="0.0"
+          iyy="1.0" iyz="0.0"
+          izz="1.0"/>
+      </inertial>
+    </link>
+    <link name="right_wheel">
+      <!--origin xyz="0.1 -0.13 0.1" rpy="0 1.5707 1.5707"/-->
+      <collision name="collision">
+        <origin xyz="0 0 0" rpy="0 1.5707 1.5707"/>
+        <geometry>
+          <cylinder radius="0.1" length="0.05"/>
+        </geometry>
+      </collision>
+      <visual name="right_wheel_visual">
+        <origin xyz="0 0 0" rpy="0 1.5707 1.5707"/>
+        <geometry>
+          <cylinder radius="0.1" length="0.05"/>
+        </geometry>
+      </visual>
+      <inertial>
+        <origin xyz="0 0 0" rpy="0 1.5707 1.5707"/>
+        <mass value="5"/>
+        <cylinder_inertia m="5" r="0.1" h="0.05"/>
+        <inertia
+          ixx="1.0" ixy="0.0" ixz="0.0"
+          iyy="1.0" iyz="0.0"
+          izz="1.0"/>
+      </inertial>
+    </link>
   <joint type="continuous" name="left_wheel_hinge">
-    <origin xyz="0.1 0.3 0" rpy="0 0 0"/>
+    <origin xyz="0.1 0.15 0" rpy="0 0 0"/>
     <child link="left_wheel"/>
     <parent link="chassis"/>
@@ -111,5 +108,5 @@
   </joint>
   <joint type="continuous" name="right_wheel_hinge">
-    <origin xyz="0.1 -0.3 0" rpy="0 0 0"/>
+    <origin xyz="0.1 -0.15 0" rpy="0 0 0"/>
     <child link="right_wheel"/>
     <parent link="chassis"/>
@@ -118,38 +115,38 @@
     <joint_properties damping="0.0" friction="0.0"/>
   </joint>
-<!--
   <link name="camera">
-    <collision>
-      <origin xyz="0 0 0" rpy="0 0 0"/>
-      <geometry>
-        <box size="${cameraSize} ${cameraSize} ${cameraSize}"/>
-      </geometry>
-    </collision>
-    <visual>
-      <origin xyz="0 0 0" rpy="0 0 0"/>
-      <geometry>
-        <box size="${cameraSize} ${cameraSize} ${cameraSize}"/>
-      </geometry>
-      <material name="green"/>
-    </visual>
-    <inertial>
-      <mass value="${cameraMass}" />
-      <origin xyz="0 0 0" rpy="0 0 0"/>
-      <box_inertia m="${cameraMass}" x="${cameraSize}" y="${cameraSize}" z="${cameraSize}" />
-      <inertia ixx="1e-6" ixy="0" ixz="0" iyy="1e-6" iyz="0" izz="1e-6" />
-    </inertial>
-  </link>
-  <joint name="camera_joint" type="fixed">
+  <collision>
+    <origin xyz="0 0 0" rpy="0 0 0"/>
+    <geometry>
+      <box size="${cameraSize} ${cameraSize} ${cameraSize}"/>
+    </geometry>
+  </collision>
+  <visual>
+    <origin xyz="0 0 0" rpy="0 0 0"/>
+    <geometry>
+      <box size="${cameraSize} ${cameraSize} ${cameraSize}"/>
+    </geometry>
+    <material name="green"/>
+  </visual>
+  <inertial>
+    <mass value="${cameraMass}" />
+    <origin xyz="0 0 0" rpy="0 0 0"/>
+    <box_inertia m="${cameraMass}" x="${cameraSize}" y="${cameraSize}" z="${cameraSize}" />
+    <inertia ixx="1e-6" ixy="0" ixz="0" iyy="1e-6" iyz="0" izz="1e-6" />
+  </inertial>
+</link>
+<joint name="camera_joint" type="fixed">
+  <axis xyz="0 1 0" />
+  <origin xyz=".2 0 0" rpy="0 0 0"/>
+  <parent link="chassis"/>
+  <child link="camera"/>
+</joint>
+  <joint name="hokuyo_joint" type="fixed">
     <axis xyz="0 1 0" />
-    <origin xyz=".2 0 0" rpy="0 0 0"/>
+    <origin xyz=".15 0 .1" rpy="0 0 0"/>
     <parent link="chassis"/>
-    <child link="camera"/>
+    <child link="hokuyo"/>
   </joint>
-  <joint name="hokuyo_joint" type="fixed">
-      <axis xyz="0 1 0" />
-      <origin xyz=".15 0 .1" rpy="0 0 0"/>
-      <parent link="chassis"/>
-      <child link="hokuyo"/>
-  </joint>
+  <!-- Hokuyo Laser -->
   <link name="hokuyo">
     <collision>
@@ -171,4 +168,3 @@
     </inertial>
   </link>
--->
 </robot>
